File: hardware/knxduino-one/knxhome.sch (EAGLE design)
At the start: 40 parts, among them U1 AP2114H-3.3TRG1, U2 STM32F334K8T6

Commit message: Switching to STM32L4 LQFP48, new TX and RX design
Parts:
- removed D12: 1N4148, diode:DIODE-MINIMELF
- removed D3: BZX84C33, diode:ZENER-DIODESOT23
- removed DEBUG: (no value), SparkFun-Connectors:CONN_03X22X3_SILK_MALE_PTH
- removed J1: (no value), SparkFun-Connectors:I2C_STANDARD
- removed JP1: (no value), pinhead:PINHD-2X10
- removed L2: 150mH, inductor-neosid:BS11
- removed LSP1: SE14, solpad:SE14
- removed SJ1, SJ2: (no value), jumper:SJ
- removed TP1, TP2, TP3, TP4: TPSQPAD1-20Y, testpad:TPSQPAD1-20Y
- removed U$1: WAGO-243-211, Connector_for_Selfbus-Projects:WAGO-243-211
- removed U1: AP2114H-3.3TRG1, ics:AP2114HWAVE-SOLDER
- removed U2: STM32F334K8T6, micro-stm_v3:STM32F334K8T6
- added BT: (no value), jumper:SJ
- added C11, C14, C15: 10u, rcl:C-EUC0805
- added C12, C16: 100n, rcl:C-EUC0805
- added C13: 10n, rcl:C-EUC0805
- added D4: 3V3, diode:ZENER-DIODESOT23
- added D5: 7V5@400mA, diode:ZENER-DIODESMB
- added D6: 400mA, zetex:DSOD323
- added DBG: (no value), SparkFun-Connectors:CONN_07LOCK
- added I2C: (no value), SparkFun-Connectors:CONN_04JST-PTH-VERT
- added I2C_U: (no value), jumper:SJ2W
- added IC1: STM32L431CCT, micro-stm_v3:STM32L051C8T
- added IOA: (no value), SparkFun-Connectors:CONN_10X2
- added IOB, IOC: (no value), SparkFun-Connectors:CONN_02
- added KNX: WAGO-243-211, Connector_for_Selfbus-Projects:WAGO-243-211
- added L3: 150mH, inductor-neosid:SD12BS11_LIEGEND
- added LED1: (no value), led:LED3MM
- added PROG: DTSM-3, switch-tact:DTSM-3
- added R10: 510R, rcl:R-EU_R0805
- added R9: 1k, rcl:R-EU_R0805
- added U3: VXO7803-500, VXO7803-500:VXO7803-500
- added U4: VXO7805-500, VXO7803-500:VXO7803-500
- C10: value 47n -> 10p
- C7: value 4u7 -> 10u
- C8: value 4u7 -> 100n
- D11: value 1N4148 -> TS4148; device diode:DIODE-MINIMELF -> diode:DIODE-D0805
- D2: value BZX84C3V3 -> 3V3
- R4: value 47k -> 33k
- R5: value 100k (NC) -> 1k
- R6: value 100k -> 0.25R
- R7: value 1k -> 100k
- R8: value 22k -> 33k
- U$2: value ROF-78E5.0-0.5SMD-R -> STCS1; device rof-78e:ROF-78E5.0-0.5SMD-R -> Synapseware:STCS1
Connections:
- removed net DCDC_OUT: C7.1, U$2.VOUT, U1.VIN
- removed net EIB+: D1.C, D11.A, D12.A, U$1.1+
- removed net EIB_AC: C10.1, D12.C, R6.2
- removed net EIB_DC: C9.+, D3.C, L2.2, U$2.VIN
- removed net KNX_RX: D2.C, R4.1, R5.2, R7.1, R7.2, R8.1, U2MCU.PB0
- removed net N$53: D11.C, L2.1
- removed net OSC_IN: C5.2, Q1.1, U2MCU.OSC_IN
- removed net OSC_OUT: C4.1, Q1.2, U2MCU.OSC_OUT
- removed net SWO: U2MCU.PB3
- removed net UART1_RX: DEBUG.3, U2MCU.PA10
- removed net UART1_TX: DEBUG.4, U2MCU.PA9
- new net +5V: C7.1, I2C_U.1, IOA.13, U4.+VOUT/GND
- new net DRX: DBG.6, IC1MCU.PA10
- new net DTX: DBG.7, IC1MCU.PA9
- new net I2C_VDD: I2C.3, I2C_U.2, IOA.18
- new net IO1: IC1MCU.PA11, IOA.1
- new net IO10: IC1MCU.PB3, IOB.2
- new net IO11: IC1MCU.PB4, IOC.2
- new net IO12: IC1MCU.PB5, IOC.1
- new net IO2: IC1MCU.PA8, IOA.2
- new net IO3: IC1MCU.PB15, IOA.4
- new net IO4: IC1MCU.PB2, IOA.6
- new net IO5: IC1MCU.PB0, IOA.8
- new net IO6: IC1MCU.PA7, IOA.9
- new net IO7: IC1MCU.PA6, IOA.10
- new net IO8: IC1MCU.PA5, IOA.12
- new net IO9: IC1MCU.PA15, IOB.1
- new net IO_RE: IC1MCU.PB1, IOA.7
- new net IO_RX: IC1MCU.PB11, IOA.3
- new net IO_TX: IC1MCU.PB10, IOA.5
- new net KNX+: D1.C, D11.A, D6.A, IOA.14, KNX.1+
- new net KNX_DC: C11.1, C14.1, C9.+, IOA.16, L3.2, R8.2, U3.+VIN, U4.+VIN
- new net KNX_DC_AN: C13.1, D2.C, IC1MCU.PA4, R8.1, R9.2
- new net KNX_RECT: C12.1, D5.C, D6.C, R4.2, U$2.EN, U$2.VCC
- new net KNX_RX_AN: C10.1, D4.C, IC1MCU.PA1, R4.1, R5.2
- new net N$3: R6.2, U$2.FB
- new net N$4: LED1.C, R10.1
- new net N$5: IC1MCU.PA0, IC1MCU.PA2
- new net N$7: C4.1, IC1MCU.OSC_OUT, Q1.1
- new net N$8: C5.2, IC1MCU.OSC_IN, Q1.2
- new net REF: D5.A, U$2.DRAIN
- net +3V3: now also BT.2, C15.1, C16.1, DBG.3, I2C_U.3, IC1PWR.VDD@1, IC1PWR.VDD@2, IC1PWR.VDD@3, IC1PWR.VDD@4, IOA.11, PROG.2, U3.+VOUT/GND; no longer DEBUG.2, J1.2, R8.2, SJ1.2, U1.VOUT, U2PWR.VDD@1, U2PWR.VDD@2
- net BOOT0: now also BT.1, IC1MCU.BOOT0; no longer SJ1.1, U2MCU.BOOT0
- net BTN: now also IC1MCU.PA12, PROG.1; no longer U2MCU.PB1
- net GND: now also C10.2, C11.2, C12.2, C13.2, C14.2, C15.2, C16.2, D4.A, DBG.4, I2C.4, IC1MCU.VSSA, IC1PWR.VSS@1, IC1PWR.VSS@2, IC1PWR.VSS@3, IOA.15, IOA.17, KNX.2-, R10.2, R7.1, R9.1, U3.GND/-VOUT, U4.GND/-VOUT; no longer D3.A, DEBUG.1, J1.1, SJ2.1, U$1.2-, U1.GND, U2PWR.VSS@1, U2PWR.VSS@2
- net I2C_SCL: now also I2C.1, IC1MCU.PB13, IOA.19; no longer J1.4, U2MCU.PB6
- net I2C_SDA: now also I2C.2, IC1MCU.PB14, IOA.20; no longer J1.3, U2MCU.PB7
- net KNX_TX: now also IC1MCU.PA3, R7.2, U$2.PWM; no longer U2MCU.PA7
- net LED: now also IC1MCU.PB12, LED1.A; no longer U2MCU.PB5
- net N$1: now also D11.C, L3.1; no longer C10.2, R4.2
- net NRST: now also DBG.1, IC1MCU.NRST; no longer SJ2.2, U2MCU.NRST
- net SWCLK: now also DBG.2, IC1MCU.PA14; no longer DEBUG.6, U2MCU.PA14
- net SWDIO: now also DBG.5, IC1MCU.PA13; no longer DEBUG.5, U2MCU.PA13
- net VDDA: no longer U2MCU.VDDA
Other:
- note added: "Calc divider in order to match KNX spec. hysteresis to COMP's selectable hysteresis"
- note removed: "2x MOSFET pro LED pasek (musel by byt optoizolovany!) radek pinu pro prime pripojeni LED pasku CW+WW (musel by byt optoizolovany!) 3x R pro primou LED (napr. RGB) xxx vstup 12v pres nizkoztratovou diodu z barel konektoru Aspon nektere vstupy/vystupy pres ochrany resistor (prinejhorim osazen 0R)"
- note removed: "Misto krystalu +2C pouzit Murata Ceralock Na Arduiny byvaji CSTCE16M0V53-R0 ale to je jen .5%, lepe presnejsi neco jako? CSTCE8M00GH5L99-R0 ST doporucuje CSTCE8M00G55-R0 nebo CSTCE8M00G15L99-R0 tento je ale uz end-of-life, ale jinak OK (.1%), ale jsou i lepsi https://cz.mouser.com/Passive-Components/Frequency-Control-Timing-Devices/Resonators/_/N-6zu9h?P=1z0wo7xZ1yx5aqg&Ns=Pricing%7c0"
- note removed: "Nahradit za integrovany oscilator TCXO?"
- note removed: "Vytahnout SWO a RESET na na debug pinheader?"
- note removed: "pridat moznost prepojit lin. regulator rovnou na 36V"
- note removed: "pridat reset (kdyby treba NRF melo programovat STMko, aby ho mohlo resetovat)"
- moved on the sheet: C1, C10, C2, C4, C5, C7, C8, C9, D1, D11, D2, L1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

Commit message: Some HW notes after first physical PCBs were made
Parts:
- C15, C7: value 10u -> 22u
- renumbered C10 to C10*, C13 to C13*, D2 to D2*, D4 to D4*
Connections:
- net VDDA: now also IC1MCU.VDDA
Other:
- note added: "Consider using LM5165 simple DC-DC for 3V3 power. Probably ignore 5V power, usually not needed (except CO2 sensors?)"
- note added: "Consider using STM32G0 + only 1 power rail (and decoupling C) + accurate internal RC (HSI), thus Xtal probably not neccessary, enabling LQFP32 package (that has no HSE)"
- note added: "Consider using logic-level mosfet + 1Watt 68R for TX +GATE-10k-GND (keep off when floating) +TX-100nF-GATE (do not allow long-time on - would be destructive to R) (simpler design, cheaper)"
- note added: "Known issues: Use switch with longer leads (adjust PCB)? no necessary. 0805 diodes are quite expensive (uncommon)! Bigger package for current sensing R! Bigger package for 10u C and 22uF at DCDC! Ferite bead peads are too small Make STCS1 pads longer for hand soldering Bigger radius place for 100uF and/or consider using SMD version Make PCB bigger in order to better fit into ITALTRONIC KNX BOX. C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"
- moved on the sheet: D11
