File: hw-design/knxduino-one/knxhome-lqfp32-v3.sch (EAGLE design)
At the start: 44 parts, among them IC1 LDL1117S33, IC3 BD9G101, IC4 STM32G071KBT6, P1 B10B-PH-K, P2 B10B-PH-K, P3 B6B-PH-K, U1 OSCILLATOR5X3-PIN1-INDICATED

Commit message: STM32G071 LQFP32 design v1.0
Parts:
- removed C10*: 10p, rcl:C-EUC0805
- removed C12: 100n, rcl:C-EUC0805
- removed C13: 4u7, rcl:C-EUC0805
- removed C16: 270n, rcl:C-EUC0805
- removed C17: 15nF, rcl:C-EUC0805
- removed D100: MBRS1100, diode:MBRA340T3
- removed IC3: BD9G101, Stefan_selfbus:BD9G101GBD9G101G-SOT23-6
- removed L2: 6.8µH, Stefan_selfbus:IND_FASTRON_1616FPS
- removed R25: 2k4, rcl:R-EU_R0805
- removed R26: 680R, rcl:R-EU_R0805
- removed U$1: ROF-78E5.0-0.5SMD-R, rof-78e:ROF-78E5.0-0.5SMD-R
- added C2', C3': *, rcl:C-EUC1210
- added C3: 22µ/10V, rcl:C-EUC1210
- added C4: 100uF 50V, rcl:CPOL-EUE3.5-8
- added C4': (no value), resistor:CPOL-EU153CLV-0810
- added C7: 1u, rcl:C-EUC0805
- added I2CB_U: (no value), jumper:SJ2W
- added LED2, RX, TX: *, led:LEDCHIPLED_1206
- added R1, R8, R9: 510R*, rcl:R-EU_R0805
- added R11, R12: 10k, rcl:R-EU_R0805
- added RX., TX.: (no value), pinhead:PINHD-1X1
- added U2: VXO7803-500, VXO7803-500:VXO7803-500
- C10: value 1u -> 10p*
- C2: value 4.7µF/50V -> 10µF/50V; device rcl:C-EUC0805 -> rcl:C-EUC1210
- C8: value 22µ/10V -> 4u7
- C9: value 100uF 50V -> 100n; device rcl:CPOL-EUE3.5-8 -> rcl:C-EUC0805
- D11: device diode:DIODE-D0805 -> diode:DIODE-SOD123
- D4: value 3V3 -> 3V3*
- D6: device zetex:DSOD323 -> diode:DIODE-SOD123
- LED1: device led:LEDCHIP-LED0805 -> led:LEDCHIPLED_1206
- renumbered D4* to D4
Connections:
- removed net ADJ: C16.1, IC3.ADJ, R25.1, R26.2
- removed net LX: C17.1, D100.C, IC3.OUT, L2.1
- removed net N$19: C17.2, IC3.BST
- removed net N$5: IC4.PA0, IC4.PA2
- new net I2C_PUP1: I2CB_U.2, R11.2, R12.2
- new net KNX_RX: IC4.PA0, IC4.PA2, RX..1, RX.C
- new net N$3: R1.2, TX.C
- new net N$4: R8.1, RX.A
- new net N$6: LED2.C, R9.2
- net +3V3: now also C8.1, I2CB_U.3, R8.2; no longer C13.1
- net GND: now also C2'.1, C3'.1, C3.1, C4'.-, C4.-, C7.2, C8.2, R1.1, R9.1, U2.GND/-VOUT; no longer C10*.2, C13.2, C8.1, C9.-, D100.A, IC3.GND, R26.1
- net I2CB_SCL: now also R11.1
- net I2CB_SDA: now also R12.1
- net IO_PB3: now also LED2.A
- net KNX_DC: now also C2'.2, C4'.+, C4.+, U2.+VIN; no longer C9.+, IC3.EN, IC3.IN
- net KNX_RX_AN: now also C10.1; no longer C10*.1
- net KNX_TX: now also C9.1, TX..1, TX.A; no longer C12.1
- net N$8: now also C9.2; no longer C12.2
- net VCC: now also C3'.2, C3.2, C7.1, I2CB_U.1, U2.+VOUT/GND; no longer C10.1, C16.2, C8.2, L2.2, R25.2
Other:
- note added: "Either: +5V line supplied Connect external +5V (3rd wire)"
- note added: "Known issues: 0805 diodes are quite expensive (uncommon)! Make PCB bigger in order to better fit into ITALTRONIC KNX BOX. Revise D6 and D11 packages RGB LEDs wont work with 3v3 power supply"
- note added: "Note: PC13, PC14 and PC15 cannot be used as current source"
- note added: "Optional: Debug LEDs"
- note removed: "Either: +5V line supplied Connect external +5V (3rd wire) to KNX_DC signal (eg. unpopulated L3's hole)"
- note removed: "Known issues: 0805 diodes are quite expensive (uncommon)! Make PCB bigger in order to better fit into ITALTRONIC KNX BOX."
- moved on the sheet: C10, C2, C8, IC1
